Commit message: add move pkg

File: src/manipulator/urdf/manipulator.urdf (robot description, URDF)
Before this commit: robot manipulator, 15 links, 14 joints
Joints:
- removed joint ÈžÀü 48
- removed joint ÈžÀü 50
- removed joint ÈžÀü 52
- removed joint ÈžÀü 54
- removed joint ÈžÀü 56
- removed joint ÈžÀü 59
- added joint motor1: type continuous, parent case1_1, child link1_1, origin xyz=-0.01425 0.028 0.013 rpy=0 0 0, axis 0.0 0.0 1.0
- added joint motor2: type continuous, parent case2_1, child link2_1, origin xyz=0.025 0.01425 0.028 rpy=0 0 0, axis 1.0 -0.0 -0.0
- added joint motor3: type continuous, parent case3_1, child link3_1, origin xyz=-0.013 0.008 0.03525 rpy=0 0 0, axis -1.0 0.0 0.0
- added joint motor4: type continuous, parent case4_1, child link4_1, origin xyz=0.028 0.01425 0.013 rpy=0 0 0, axis 0.0 0.0 1.0
- added joint motor5: type continuous, parent case5_1, child link5_1, origin xyz=0.013 -0.01425 0.004 rpy=0 0 0, axis 1.0 -0.0 -0.0
- added joint motor6: type continuous, parent case6_1, child link7_1, origin xyz=-0.008 -0.025 0.03525 rpy=0 0 0, axis -0.0 -1.0 -0.0
